File: main_board/kicad/bridge.kicad_sch (KiCad schematic)
At the start: 21 parts, among them Q1 IRFB3077, Q2 IRFB3077, Q3 IRFB3077, Q4 IRFB3077, Q5 IRFB3077, Q6 IRFB3077

Commit message: revamped root and bridge
Connections:
- net Y_OUT renamed V_OUT3
