File: main_board/kicad/bridgeDriver.kicad_sch (KiCad schematic)
At the start: 1 part, among them U3 IR2133

Commit message: bridge driver almost done
Parts:
- added C10, C6, C7, C8, C9: C_Polarized, symbol Device:C_Polarized
- added D2, D3, D4: D, symbol Device:D
- added R4, R5, R6, R7, R8, R9: R, symbol Device:R
Connections:
- net at U3.10 (LO2): now also R8.1
- net at U3.11 (LO1): now also R7.1
- net VS3: now reaches U3.12 (VS3)
- net VS3: now also C7.2, C8.2
- net at U3.13 (HO3): now also R6.1
- net at U3.14 (VB3): now also C8.1, D4.1 (K)
- net VS2: now reaches U3.15 (VS2)
- net at U3.16 (HO2): now also R5.1
- net at U3.17 (VB2): now also C7.1, D3.1 (K)
- net VS1: now reaches U3.18 (VS1)
- net VS1: now also C6.2
- net at U3.19 (HO1): now also R4.1
- net at U3.20 (VB1): now also C6.1, D2.1 (K)
- net +15V: now reaches U3.21 (VCC)
- net +15V: now also U3.7 (VSS), U3.8 (COM), C10.1, C10.2, C9.1, C9.2, D2.2 (A), D3.2 (A), D4.2 (A)
- net HIN1: now reaches U3.22 (~{HIN1})
- net HIN2: now reaches U3.23 (~{HIN2})
- net HIN3: now reaches U3.24 (~{HIN3})
- net LIN1: now reaches U3.25 (~{LIN1})
- net LIN2: now reaches U3.26 (~{LIN2})
- net LIN3: now reaches U3.27 (~{LIN3})
- net at U3.9 (LO3): now also R9.1
- new net HO1: R4.2
- new net HO2: R5.2
- new net HO3: R6.2
- new net LO1: R7.2
- new net LO2: R8.2
- new net LO3: R9.2

Commit message: added communication logic
Connections:
- net HIN1 renamed B_H_IN
- net HIN2 renamed G_H_IN
- net HIN3 renamed Y_H_IN
- net HO1 renamed B_H_OUT
- net HO2 renamed G_H_OUT
- net HO3 renamed Y_H_OUT
- net LIN1 renamed B_L_IN
- net LIN2 renamed G_L_IN
- net LIN3 renamed Y_L_IN
- net LO1 renamed B_L_OUT
- net LO2 renamed G_L_OUT
- net LO3 renamed Y_L_OUT
Changed lines of the file:
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@@
     (stroke (width 0) (type default))
   )
-  (hierarchical_label "HIN1" (shape input) (at 123.19 87.63 180) (fields_autoplaced)
+  (hierarchical_label "B_H_IN" (shape input) (at 123.19 87.63 180) (fields_autoplaced)
     (effects (font (size 1.27 1.27)) (justify right))
   )
-  (hierarchical_label "HO3" (shape input) (at 203.2 80.01 0) (fields_autoplaced)
+  (hierarchical_label "Y_H_OUT" (shape output) (at 203.2 80.01 0) (fields_autoplaced)
     (effects (font (size 1.27 1.27)) (justify left))
   )
-  (hierarchical_label "HIN3" (shape input) (at 123.19 92.71 180) (fields_autoplaced)
+  (hierarchical_label "Y_H_IN" (shape input) (at 123.19 92.71 180) (fields_autoplaced)
     (effects (font (size 1.27 1.27)) (justify right))
   )
-  (hierarchical_label "VS1" (shape input) (at 203.2 95.25 0) (fields_autoplaced)
+  (hierarchical_label "VS1" (shape output) (at 203.2 95.25 0) (fields_autoplaced)
     (effects (font (size 1.27 1.27)) (justify left))
   )
-  (hierarchical_label "LIN1" (shape input) (at 123.19 95.25 180) (fields_autoplaced)
+  (hierarchical_label "B_L_IN" (shape input) (at 123.19 95.25 180) (fields_autoplaced)
     (effects (font (size 1.27 1.27)) (justify right))
   )
-  (hierarchical_label "HIN2" (shape input) (at 123.19 90.17 180) (fields_autoplaced)
+  (hierarchical_label "G_H_IN" (shape input) (at 123.19 90.17 180) (fields_autoplaced)
     (effects (font (size 1.27 1.27)) (justify right))
   )
-  (hierarchical_label "LIN2" (shape input) (at 123.19 97.79 180) (fields_autoplaced)
+  (hierarchical_label "G_L_IN" (shape input) (at 123.19 97.79 180) (fields_autoplaced)
     (effects (font (size 1.27 1.27)) (justify right))
   )
-  (hierarchical_label "VS2" (shape input) (at 203.2 102.87 0) (fields_autoplaced)
+  (hierarchical_label "VS2" (shape output) (at 203.2 102.87 0) (fields_autoplaced)
     (effects (font (size 1.27 1.27)) (justify left))
   )
-  (hierarchical_label "HO2" (shape input) (at 203.2 72.39 0) (fields_autoplaced)
+  (hierarchical_label "G_H_OUT" (shape output) (at 203.2 72.39 0) (fields_autoplaced)
     (effects (font (size 1.27 1.27)) (justify left))
   )
-  (hierarchical_label "LO1" (shape input) (at 203.2 125.73 0) (fields_autoplaced)
+  (hierarchical_label "B_L_OUT" (shape output) (at 203.2 125.73 0) (fields_autoplaced)
     (effects (font (size 1.27 1.27)) (justify left))
   )
-  (hierarchical_label "VS3" (shape input) (at 203.2 110.49 0) (fields_autoplaced)
+  (hierarchical_label "VS3" (shape output) (at 203.2 110.49 0) (fields_autoplaced)
     (effects (font (size 1.27 1.27)) (justify left))
   )
-  (hierarchical_label "LIN3" (shape input) (at 123.19 100.33 180) (fields_autoplaced)
+  (hierarchical_label "Y_L_IN" (shape input) (at 123.19 100.33 180) (fields_autoplaced)
     (effects (font (size 1.27 1.27)) (justify right))
   )
-  (hierarchical_label "LO3" (shape input) (at 203.2 140.97 0) (fields_autoplaced)
+  (hierarchical_label "Y_L_OUT" (shape output) (at 203.2 140.97 0) (fields_autoplaced)
     (effects (font (size 1.27 1.27)) (justify left))
   )
-  (hierarchical_label "HO1" (shape input) (at 203.2 64.77 0) (fields_autoplaced)
+  (hierarchical_label "B_H_OUT" (shape output) (at 203.2 64.77 0) (fields_autoplaced)
     (effects (font (size 1.27 1.27)) (justify left))
   )
-  (hierarchical_label "LO2" (shape input) (at 203.2 133.35 0) (fields_autoplaced)
+  (hierarchical_label "G_L_OUT" (shape output) (at 203.2 133.35 0) (fields_autoplaced)
     (effects (font (size 1.27 1.27)) (justify left))
   )

Commit message: huh
Parts:
- added R23: R, symbol Device:R
Connections:
- net /ENABLE: now reaches U3.6 (SD)
- net /ENABLE: now also R23.2
- new net +5V: R23.1
Changed lines of the file:
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@@
   (junction (at 152.4 81.28) (diameter 0) (color 0 0 0 0)
   )
+  (junction (at 102.87 110.49) (diameter 0) (color 0 0 0 0)
+  )
   (junction (at 144.78 81.28) (diameter 0) (color 0 0 0 0)
   )
@@
     (stroke (width 0) (type default))
   )
+  (wire (pts (xy 102.87 109.22) (xy 102.87 110.49))
+    (stroke (width 0) (type default))
+  )
   (wire (pts (xy 111.76 128.27) (xy 133.35 128.27))
     (stroke (width 0) (type default))
@@
     (stroke (width 0) (type default))
   )
+  (wire (pts (xy 102.87 110.49) (xy 123.19 110.49))
+    (stroke (width 0) (type default))
+  )
   (wire (pts (xy 143.51 97.79) (xy 163.83 97.79))
     (stroke (width 0) (type default))
@@
   )
   (wire (pts (xy 144.78 76.2) (xy 144.78 81.28))
+    (stroke (width 0) (type default))
+  )
+  (wire (pts (xy 88.9 110.49) (xy 102.87 110.49))
     (stroke (width 0) (type default))
   )
@@
     (effects (font (size 1.27 1.27)) (justify right))
   )
+  (hierarchical_label "{slash}ENABLE" (shape input) (at 88.9 110.49 180) (fields_autoplaced)
+    (effects (font (size 1.27 1.27)) (justify right))
+  )
   (hierarchical_label "Y_H_OUT" (shape output) (at 203.2 80.01 0) (fields_autoplaced)
     (effects (font (size 1.27 1.27)) (justify left))
@@
         (path "/9139d8e7-a5dc-421f-9a12-f77d83384a16/f375863d-6ceb-4c75-8514-48e21c11bcc5"
           (reference "#PWR018") (unit 1)
+        )
+        (path "/9139d8e7-a5dc-421f-9a12-f77d83384a16/9bcba079-9422-42f1-a7c0-49fe4d0b5e5a"
+          (reference "#PWR037") (unit 1)
         )
       )
@@
           (reference "U3") (unit 1)
         )
+        (path "/9139d8e7-a5dc-421f-9a12-f77d83384a16/9bcba079-9422-42f1-a7c0-49fe4d0b5e5a"
+          (reference "U6") (unit 1)
+        )
       )
     )
@@
           (reference "R5") (unit 1)
         )
+        (path "/9139d8e7-a5dc-421f-9a12-f77d83384a16/9bcba079-9422-42f1-a7c0-49fe4d0b5e5a"
+          (reference "R11") (unit 1)
+        )
       )
     )
@@
           (reference "#PWR017") (unit 1)
         )
+        (path "/9139d8e7-a5dc-421f-9a12-f77d83384a16/9bcba079-9422-42f1-a7c0-49fe4d0b5e5a"
+          (reference "#PWR038") (unit 1)
+        )
       )
     )
@@
           (reference "R4") (unit 1)
         )
+        (path "/9139d8e7-a5dc-421f-9a12-f77d83384a16/9bcba079-9422-42f1-a7c0-49fe4d0b5e5a"
+          (reference "R10") (unit 1)
+        )
       )
     )
@@
           (reference "C8") (unit 1)
         )
+        (path "/9139d8e7-a5dc-421f-9a12-f77d83384a16/9bcba079-9422-42f1-a7c0-49fe4d0b5e5a"
+          (reference "C23") (unit 1)
+        )
+      )
+    )
+  )
+  (symbol (lib_id "Device:R") (at 102.87 105.41 0) (unit 1)
+    (in_bom yes) (on_board yes) (dnp no) (fields_autoplaced)
+    (property "Reference" "R23" (at 105.41 104.14 0)
+      (effects (font (size 1.27 1.27)) (justify left))
+    )
+    (property "Value" "R" (at 105.41 106.68 0)
+      (effects (font (size 1.27 1.27)) (justify left))
+    )
+    (property "Footprint" "" (at 101.092 105.41 90)
+      (effects (font (size 1.27 1.27)) hide)
+    )
+    (property "Datasheet" "~" (at 102.87 105.41 0)
+      (effects (font (size 1.27 1.27)) hide)
+    )
+    (pin "1")
+    (pin "2")
+    (instances
+      (project "main"
+        (path "/9139d8e7-a5dc-421f-9a12-f77d83384a16/9bcba079-9422-42f1-a7c0-49fe4d0b5e5a"
+          (reference "R23") (unit 1)
+        )
+        (path "/9139d8e7-a5dc-421f-9a12-f77d83384a16/f375863d-6ceb-4c75-8514-48e21c11bcc5"
+          (reference "R22") (unit 1)
+        )
       )
     )
@@
         (path "/9139d8e7-a5dc-421f-9a12-f77d83384a16/f375863d-6ceb-4c75-8514-48e21c11bcc5"
           (reference "C9") (unit 1)
+        )
+        (path "/9139d8e7-a5dc-421f-9a12-f77d83384a16/9bcba079-9422-42f1-a7c0-49fe4d0b5e5a"
+          (reference "C19") (unit 1)
         )
       )
@@
           (reference "C6") (unit 1)
         )
+        (path "/9139d8e7-a5dc-421f-9a12-f77d83384a16/9bcba079-9422-42f1-a7c0-49fe4d0b5e5a"
+          (reference "C21") (unit 1)
+        )
       )
     )
@@
           (reference "D3") (unit 1)
         )
+        (path "/9139d8e7-a5dc-421f-9a12-f77d83384a16/9bcba079-9422-42f1-a7c0-49fe4d0b5e5a"
+          (reference "D7") (unit 1)
+        )
       )
     )
@@
         (path "/9139d8e7-a5dc-421f-9a12-f77d83384a16/f375863d-6ceb-4c75-8514-48e21c11bcc5"
           (reference "D4") (unit 1)
+        )
+        (path "/9139d8e7-a5dc-421f-9a12-f77d83384a16/9bcba079-9422-42f1-a7c0-49fe4d0b5e5a"
+          (reference "D8") (unit 1)
         )
       )
@@
           (reference "C7") (unit 1)
         )
+        (path "/9139d8e7-a5dc-421f-9a12-f77d83384a16/9bcba079-9422-42f1-a7c0-49fe4d0b5e5a"
+          (reference "C22") (unit 1)
+        )
+      )
+    )
+  )
+  (symbol (lib_id "power:+5V") (at 102.87 101.6 0) (unit 1)
+    (in_bom yes) (on_board yes) (dnp no) (fields_autoplaced)
+    (property "Reference" "#PWR049" (at 102.87 105.41 0)
+      (effects (font (size 1.27 1.27)) hide)
+    )
+    (property "Value" "+5V" (at 102.87 96.52 0)
+      (effects (font (size 1.27 1.27)))
+    )
+    (property "Footprint" "" (at 102.87 101.6 0)
+      (effects (font (size 1.27 1.27)) hide)
+    )
+    (property "Datasheet" "" (at 102.87 101.6 0)
+      (effects (font (size 1.27 1.27)) hide)
+    )
+    (pin "1")
+    (instances
+      (project "main"
+        (path "/9139d8e7-a5dc-421f-9a12-f77d83384a16/9bcba079-9422-42f1-a7c0-49fe4d0b5e5a"
+          (reference "#PWR049") (unit 1)
+        )
+        (path "/9139d8e7-a5dc-421f-9a12-f77d83384a16/f375863d-6ceb-4c75-8514-48e21c11bcc5"
+          (reference "#PWR048") (unit 1)
+        )
       )
     )
@@
           (reference "C10") (unit 1)
         )
+        (path "/9139d8e7-a5dc-421f-9a12-f77d83384a16/9bcba079-9422-42f1-a7c0-49fe4d0b5e5a"
+          (reference "C20") (unit 1)
+        )
       )
     )
@@
           (reference "R8") (unit 1)
         )
+        (path "/9139d8e7-a5dc-421f-9a12-f77d83384a16/9bcba079-9422-42f1-a7c0-49fe4d0b5e5a"
+          (reference "R14") (unit 1)
+        )
       )
     )
@@
           (reference "R6") (unit 1)
         )
+        (path "/9139d8e7-a5dc-421f-9a12-f77d83384a16/9bcba079-9422-42f1-a7c0-49fe4d0b5e5a"
+          (reference "R12") (unit 1)
+        )
       )
     )
@@
         (path "/9139d8e7-a5dc-421f-9a12-f77d83384a16/f375863d-6ceb-4c75-8514-48e21c11bcc5"
           (reference "R9") (unit 1)
+        )
+        (path "/9139d8e7-a5dc-421f-9a12-f77d83384a16/9bcba079-9422-42f1-a7c0-49fe4d0b5e5a"
+          (reference "R15") (unit 1)
         )
       )
@@
           (reference "D2") (unit 1)
         )
+        (path "/9139d8e7-a5dc-421f-9a12-f77d83384a16/9bcba079-9422-42f1-a7c0-49fe4d0b5e5a"
+          (reference "D6") (unit 1)
+        )
       )
     )
@@
           (reference "R7") (unit 1)
         )
-      )
+        (path "/9139d8e7-a5dc-421f-9a12-f77d83384a16/9bcba079-9422-42f1-a7c0-49fe4d0b5e5a"
+          (reference "R13") (unit 1)
+        )
+      )

Commit message: added ISP socket for attiny
Parts:
- renumbered C9 to C35, C10 to C36, C6 to C37, C7 to C38, C8 to C39, D2 to D12, D3 to D13, D4 to D14, R23 to R30, R4 to R31, R5 to R32, R6 to R33, R7 to R34, R8 to R35, R9 to R36, U3 to U9
Changed lines of the file:
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@@
   (symbol (lib_id "power:+15V") (at 107.95 63.5 0) (unit 1)
     (in_bom yes) (on_board yes) (dnp no) (fields_autoplaced)
-    (property "Reference" "#PWR018" (at 107.95 67.31 0)
+    (property "Reference" "#PWR063" (at 107.95 67.31 0)
       (effects (font (size 1.27 1.27)) hide)
     )
@@
   (symbol (lib_id "Driver_FET:IR2133") (at 133.35 105.41 0) (unit 1)
     (in_bom yes) (on_board yes) (dnp no) (fields_autoplaced)
-    (property "Reference" "U3" (at 135.5441 80.01 0)
+    (property "Reference" "U9" (at 135.5441 80.01 0)
       (effects (font (size 1.27 1.27)) (justify left))
     )
@@
   (symbol (lib_id "Device:R") (at 199.39 72.39 90) (unit 1)
     (in_bom yes) (on_board yes) (dnp no) (fields_autoplaced)
-    (property "Reference" "R5" (at 199.39 66.04 90)
+    (property "Reference" "R32" (at 199.39 66.04 90)
       (effects (font (size 1.27 1.27)))
     )
@@
   (symbol (lib_id "power:GND") (at 143.51 128.27 0) (unit 1)
     (in_bom yes) (on_board yes) (dnp no) (fields_autoplaced)
-    (property "Reference" "#PWR017" (at 143.51 134.62 0)
+    (property "Reference" "#PWR064" (at 143.51 134.62 0)
       (effects (font (size 1.27 1.27)) hide)
     )
@@
   (symbol (lib_id "Device:R") (at 199.39 64.77 90) (unit 1)
     (in_bom yes) (on_board yes) (dnp no) (fields_autoplaced)
-    (property "Reference" "R4" (at 199.39 58.42 90)
+    (property "Reference" "R31" (at 199.39 58.42 90)
       (effects (font (size 1.27 1.27)))
     )
@@
   (symbol (lib_id "Device:C_Polarized") (at 179.07 45.72 90) (unit 1)
     (in_bom yes) (on_board yes) (dnp no) (fields_autoplaced)
-    (property "Reference" "C8" (at 176.911 41.91 0)
+    (property "Reference" "C39" (at 176.911 41.91 0)
       (effects (font (size 1.27 1.27)) (justify left))
     )
@@
   (symbol (lib_id "Device:R") (at 102.87 105.41 0) (unit 1)
     (in_bom yes) (on_board yes) (dnp no) (fields_autoplaced)
-    (property "Reference" "R23" (at 105.41 104.14 0)
+    (property "Reference" "R30" (at 105.41 104.14 0)
       (effects (font (size 1.27 1.27)) (justify left))
     )
@@
   (symbol (lib_id "Device:C_Polarized") (at 111.76 124.46 0) (unit 1)
     (in_bom yes) (on_board yes) (dnp no) (fields_autoplaced)
-    (property "Reference" "C9" (at 115.57 122.301 0)
+    (property "Reference" "C35" (at 115.57 122.301 0)
       (effects (font (size 1.27 1.27)) (justify left))
     )
@@
   (symbol (lib_id "Device:C_Polarized") (at 156.21 81.28 90) (unit 1)
     (in_bom yes) (on_board yes) (dnp no)
-    (property "Reference" "C6" (at 154.051 77.47 0)
+    (property "Reference" "C37" (at 154.051 77.47 0)
       (effects (font (size 1.27 1.27)) (justify left))
     )
@@
   (symbol (lib_id "Device:D") (at 160.02 63.5 180) (unit 1)
     (in_bom yes) (on_board yes) (dnp no) (fields_autoplaced)
-    (property "Reference" "D3" (at 158.75 60.96 90)
+    (property "Reference" "D13" (at 158.75 60.96 90)
       (effects (font (size 1.27 1.27)) (justify right))
     )
@@
   (symbol (lib_id "Device:D") (at 171.45 45.72 180) (unit 1)
     (in_bom yes) (on_board yes) (dnp no) (fields_autoplaced)
-    (property "Reference" "D4" (at 170.18 43.18 90)
+    (property "Reference" "D14" (at 170.18 43.18 90)
       (effects (font (size 1.27 1.27)) (justify right))
     )
@@
   (symbol (lib_id "Device:C_Polarized") (at 167.64 63.5 90) (unit 1)
     (in_bom yes) (on_board yes) (dnp no)
-    (property "Reference" "C7" (at 165.481 59.69 0)
+    (property "Reference" "C38" (at 165.481 59.69 0)
       (effects (font (size 1.27 1.27)) (justify left))
     )
@@
   (symbol (lib_id "power:+5V") (at 102.87 101.6 0) (unit 1)
     (in_bom yes) (on_board yes) (dnp no) (fields_autoplaced)
-    (property "Reference" "#PWR049" (at 102.87 105.41 0)
+    (property "Reference" "#PWR062" (at 102.87 105.41 0)
       (effects (font (size 1.27 1.27)) hide)
     )
@@
   (symbol (lib_id "Device:C_Polarized") (at 144.78 72.39 0) (unit 1)
     (in_bom yes) (on_board yes) (dnp no) (fields_autoplaced)
-    (property "Reference" "C10" (at 148.59 70.231 0)
+    (property "Reference" "C36" (at 148.59 70.231 0)
       (effects (font (size 1.27 1.27)) (justify left))
     )
@@
   (symbol (lib_id "Device:R") (at 199.39 133.35 90) (unit 1)
     (in_bom yes) (on_board yes) (dnp no) (fields_autoplaced)
-    (property "Reference" "R8" (at 199.39 127 90)
+    (property "Reference" "R35" (at 199.39 127 90)
       (effects (font (size 1.27 1.27)))
     )
@@
   (symbol (lib_id "Device:R") (at 199.39 80.01 90) (unit 1)
     (in_bom yes) (on_board yes) (dnp no) (fields_autoplaced)
-    (property "Reference" "R6" (at 199.39 73.66 90)
+    (property "Reference" "R33" (at 199.39 73.66 90)
       (effects (font (size 1.27 1.27)))
     )
@@
   (symbol (lib_id "Device:R") (at 199.39 140.97 90) (unit 1)
     (in_bom yes) (on_board yes) (dnp no) (fields_autoplaced)
-    (property "Reference" "R9" (at 199.39 134.62 90)
+    (property "Reference" "R36" (at 199.39 134.62 90)
       (effects (font (size 1.27 1.27)))
     )
@@
   (symbol (lib_id "Device:D") (at 148.59 81.28 180) (unit 1)
     (in_bom yes) (on_board yes) (dnp no) (fields_autoplaced)
-    (property "Reference" "D2" (at 147.32 78.74 90)
+    (property "Reference" "D12" (at 147.32 78.74 90)
       (effects (font (size 1.27 1.27)) (justify right))
     )
@@
   (symbol (lib_id "Device:R") (at 199.39 125.73 90) (unit 1)
     (in_bom yes) (on_board yes) (dnp no) (fields_autoplaced)
-    (property "Reference" "R7" (at 199.39 119.38 90)
-      (effects (font (size 1.27 1.27)))
-    )
+    (property "Reference" "R34" (at 199.39 119.38 90)
+      (effects (font (size 1.27 1.27)))
+    )

Commit message: added pull up resistor values
Parts:
- R30: value R -> 50k
Changed lines of the file:
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@@
       (effects (font (size 1.27 1.27)) (justify left))
     )
-    (property "Value" "R" (at 105.41 106.68 0)
+    (property "Value" "50k" (at 105.41 106.68 0)
       (effects (font (size 1.27 1.27)) (justify left))
     )

Commit message: fixed pull up resistor values
Parts:
- R30: value 50k -> 30k
Changed lines of the file:
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@@
       (effects (font (size 1.27 1.27)) (justify left))
     )
-    (property "Value" "50k" (at 105.41 106.68 0)
+    (property "Value" "30k" (at 105.41 106.68 0)
       (effects (font (size 1.27 1.27)) (justify left))
     )
