File: main_board/kicad/bridgeDriver.kicad_sch (KiCad schematic)
At the start: 16 parts, among them U9 IR2133

Commit message: added funny fun file
Parts:
- R31: value R -> 62
Connections:
- net +15V: no longer C35.2, C36.2, U9.7 (VSS), U9.8 (COM)
- new net GND: C35.2, C36.2, U9.7 (VSS), U9.8 (COM)
Other:
- moved on the sheet: C37, C38
Changed lines of the file:
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@@
 (kicad_sch (version 20230121) (generator eeschema)
   (paper "A4")
+  (junction (at 152.4 81.28) (diameter 0) (color 0 0 0 0)
+  )
   (junction (at 133.35 81.28) (diameter 0) (color 0 0 0 0)
   )
   (junction (at 111.76 63.5) (diameter 0) (color 0 0 0 0)
   )
+  (junction (at 158.75 95.25) (diameter 0) (color 0 0 0 0)
+  )
   (junction (at 133.35 63.5) (diameter 0) (color 0 0 0 0)
   )
+  (junction (at 133.35 128.27) (diameter 0) (color 0 0 0 0)
+  )
+  (junction (at 170.18 110.49) (diameter 0) (color 0 0 0 0)
+  )
+  (junction (at 102.87 110.49) (diameter 0) (color 0 0 0 0)
+  )
+  (junction (at 144.78 63.5) (diameter 0) (color 0 0 0 0)
+  )
+  (junction (at 175.26 45.72) (diameter 0) (color 0 0 0 0)
+  )
+  (junction (at 182.88 110.49) (diameter 0) (color 0 0 0 0)
+  )
+  (junction (at 143.51 128.27) (diameter 0) (color 0 0 0 0)
+  )
   (junction (at 163.83 63.5) (diameter 0) (color 0 0 0 0)
   )
-  (junction (at 133.35 128.27) (diameter 0) (color 0 0 0 0)
-  )
-  (junction (at 171.45 110.49) (diameter 0) (color 0 0 0 0)
-  )
-  (junction (at 160.02 95.25) (diameter 0) (color 0 0 0 0)
-  )
-  (junction (at 152.4 81.28) (diameter 0) (color 0 0 0 0)
-  )
-  (junction (at 102.87 110.49) (diameter 0) (color 0 0 0 0)
-  )
-  (junction (at 144.78 81.28) (diameter 0) (color 0 0 0 0)
-  )
-  (junction (at 144.78 63.5) (diameter 0) (color 0 0 0 0)
-  )
-  (junction (at 175.26 45.72) (diameter 0) (color 0 0 0 0)
-  )
-  (junction (at 182.88 110.49) (diameter 0) (color 0 0 0 0)
-  )
-  (junction (at 143.51 128.27) (diameter 0) (color 0 0 0 0)
-  )
   (wire (pts (xy 181.61 133.35) (xy 195.58 133.35))
     (stroke (width 0) (type default))
@@
     (stroke (width 0) (type default))
   )
-  (wire (pts (xy 160.02 95.25) (xy 203.2 95.25))
-    (stroke (width 0) (type default))
-  )
-  (wire (pts (xy 160.02 81.28) (xy 160.02 95.25))
+  (wire (pts (xy 152.4 81.28) (xy 158.75 81.28))
     (stroke (width 0) (type default))
   )
@@
     (stroke (width 0) (type default))
   )
-  (wire (pts (xy 143.51 95.25) (xy 160.02 95.25))
+  (wire (pts (xy 143.51 95.25) (xy 158.75 95.25))
     (stroke (width 0) (type default))
   )
@@
     (stroke (width 0) (type default))
   )
+  (wire (pts (xy 170.18 110.49) (xy 182.88 110.49))
+    (stroke (width 0) (type default))
+  )
   (wire (pts (xy 143.51 102.87) (xy 203.2 102.87))
     (stroke (width 0) (type default))
   )
+  (wire (pts (xy 158.75 88.9) (xy 158.75 95.25))
+    (stroke (width 0) (type default))
+  )
   (wire (pts (xy 143.51 105.41) (xy 175.26 105.41))
     (stroke (width 0) (type default))
@@
     (stroke (width 0) (type default))
   )
-  (wire (pts (xy 171.45 110.49) (xy 182.88 110.49))
+  (wire (pts (xy 158.75 95.25) (xy 203.2 95.25))
     (stroke (width 0) (type default))
   )
@@
     (stroke (width 0) (type default))
   )
+  (wire (pts (xy 163.83 63.5) (xy 170.18 63.5))
+    (stroke (width 0) (type default))
+  )
   (wire (pts (xy 133.35 63.5) (xy 133.35 81.28))
     (stroke (width 0) (type default))
@@
     (stroke (width 0) (type default))
   )
-  (wire (pts (xy 144.78 76.2) (xy 144.78 81.28))
+  (wire (pts (xy 144.78 76.2) (xy 144.78 128.27))
     (stroke (width 0) (type default))
   )
@@
     (stroke (width 0) (type default))
   )
-  (wire (pts (xy 171.45 63.5) (xy 171.45 110.49))
-    (stroke (width 0) (type default))
-  )
   (wire (pts (xy 143.51 90.17) (xy 152.4 90.17))
     (stroke (width 0) (type default))
@@
     (stroke (width 0) (type default))
   )
-  (wire (pts (xy 143.51 110.49) (xy 171.45 110.49))
+  (wire (pts (xy 143.51 110.49) (xy 170.18 110.49))
     (stroke (width 0) (type default))
   )
@@
     (stroke (width 0) (type default))
   )
-  (wire (pts (xy 144.78 81.28) (xy 144.78 128.27))
-    (stroke (width 0) (type default))
-  )
   (wire (pts (xy 111.76 63.5) (xy 133.35 63.5))
+    (stroke (width 0) (type default))
+  )
+  (wire (pts (xy 170.18 71.12) (xy 170.18 110.49))
     (stroke (width 0) (type default))
   )
@@
       (effects (font (size 1.27 1.27)))
     )
-    (property "Value" "R" (at 199.39 60.96 90)
+    (property "Value" "62" (at 199.39 60.96 90)
       (effects (font (size 1.27 1.27)))
     )
@@
     )
   )
-  (symbol (lib_id "Device:C_Polarized") (at 156.21 81.28 90) (unit 1)
+  (symbol (lib_id "Device:C_Polarized") (at 158.75 85.09 0) (unit 1)
     (in_bom yes) (on_board yes) (dnp no)
-    (property "Reference" "C37" (at 154.051 77.47 0)
-      (effects (font (size 1.27 1.27)) (justify left))
-    )
-    (property "Value" "C_Polarized" (at 156.591 77.47 0)
-      (effects (font (size 1.27 1.27)) (justify left))
-    )
-    (property "Footprint" "" (at 160.02 80.3148 0)
-      (effects (font (size 1.27 1.27)) hide)
-    )
-    (property "Datasheet" "~" (at 156.21 81.28 0)
+    (property "Reference" "C37" (at 162.56 82.931 0)
+      (effects (font (size 1.27 1.27)) (justify left))
+    )
+    (property "Value" "C_Polarized" (at 162.56 85.471 0)
+      (effects (font (size 1.27 1.27)) (justify left))
+    )
+    (property "Footprint" "" (at 159.7152 88.9 0)
+      (effects (font (size 1.27 1.27)) hide)
+    )
+    (property "Datasheet" "~" (at 158.75 85.09 0)
       (effects (font (size 1.27 1.27)) hide)
     )
@@
     )
   )
-  (symbol (lib_id "Device:C_Polarized") (at 167.64 63.5 90) (unit 1)
+  (symbol (lib_id "Device:C_Polarized") (at 170.18 67.31 0) (unit 1)
     (in_bom yes) (on_board yes) (dnp no)
-    (property "Reference" "C38" (at 165.481 59.69 0)
-      (effects (font (size 1.27 1.27)) (justify left))
-    )
-    (property "Value" "C_Polarized" (at 168.021 59.69 0)
-      (effects (font (size 1.27 1.27)) (justify left))
-    )
-    (property "Footprint" "" (at 171.45 62.5348 0)
-      (effects (font (size 1.27 1.27)) hide)
-    )
-    (property "Datasheet" "~" (at 167.64 63.5 0)
-      (effects (font (size 1.27 1.27)) hide)
-    )
+    (property "Reference" "C38" (at 173.99 65.151 0)
+      (effects (font (size 1.27 1.27)) (justify left))
+    )
+    (property "Value" "C_Polarized" (at 173.99 67.691 0)
+      (effects (font (size 1.27 1.27)) (justify left))
+    )
+    (property "Footprint" "" (at 171.1452 71.12 0)
+      (effects (font (size 1.27 1.27)) hide)
+    )
+    (property "Datasheet" "~" (at 170.18 67.31 0)
+      (effects (font (size 1.27 1.27)) hide)
+    )
