File: main_board/kicad/commutationLogic.kicad_sch (KiCad schematic)
At the start: 2 parts, among them U5 AT28C64B

Commit message: huh
Parts:
- added C25, C27, C29: C, symbol Device:C
- added R16, R18, R20, R25: R, symbol Device:R
Connections:
- net +5V: now also R25.1
- net GND: now also C25.2, C27.2, C29.2; no longer U5.22 (OE)
- net HAL1: now also R16.1; no longer U5.10 (A0)
- net HAL2: now also R18.1; no longer U5.9 (A1)
- net HAL3: now also R20.1; no longer U5.8 (A2)
- new net: C27.1, R18.2, U5.9 (A1)
- new net: C25.1, R16.2, U5.10 (A0)
- new net: C29.1, R20.2, U5.8 (A2)
- new net /ENABLE: R25.2, U5.22 (OE)
- no-connect marks 5 -> 4
Other:
- moved on the sheet: C15

Commit message: added ISP socket for attiny
Parts:
- renumbered C25 to C31, C15 to C32, C27 to C33, C29 to C34, R16 to R26, R18 to R27, R20 to R28, R25 to R29, U5 to U8
Changed lines of the file:
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@@
   (symbol (lib_id "Device:R") (at 110.49 93.98 90) (unit 1)
     (in_bom yes) (on_board yes) (dnp no) (fields_autoplaced)
-    (property "Reference" "R18" (at 110.49 87.63 90)
+    (property "Reference" "R27" (at 110.49 87.63 90)
       (effects (font (size 1.27 1.27)))
     )
@@
   (symbol (lib_id "power:+5V") (at 106.68 134.62 0) (unit 1)
     (in_bom yes) (on_board yes) (dnp no) (fields_autoplaced)
-    (property "Reference" "#PWR025" (at 106.68 138.43 0)
+    (property "Reference" "#PWR055" (at 106.68 138.43 0)
       (effects (font (size 1.27 1.27)) hide)
     )
@@
   (symbol (lib_id "2022-lsd:AT28C64B") (at 148.59 99.06 0) (unit 1)
     (in_bom yes) (on_board yes) (dnp no) (fields_autoplaced)
-    (property "Reference" "U5" (at 148.59 76.2 0)
+    (property "Reference" "U8" (at 148.59 76.2 0)
       (effects (font (size 1.27 1.27)))
     )
@@
   (symbol (lib_id "Device:R") (at 179.07 95.25 0) (unit 1)
     (in_bom yes) (on_board yes) (dnp no) (fields_autoplaced)
-    (property "Reference" "R25" (at 181.61 93.98 0)
+    (property "Reference" "R29" (at 181.61 93.98 0)
       (effects (font (size 1.27 1.27)) (justify left))
     )
@@
   (symbol (lib_id "Device:R") (at 121.92 82.55 90) (unit 1)
     (in_bom yes) (on_board yes) (dnp no) (fields_autoplaced)
-    (property "Reference" "R20" (at 121.92 76.2 90)
+    (property "Reference" "R28" (at 121.92 76.2 90)
       (effects (font (size 1.27 1.27)))
     )
@@
   (symbol (lib_id "power:GND") (at 106.68 142.24 0) (unit 1)
     (in_bom yes) (on_board yes) (dnp no) (fields_autoplaced)
-    (property "Reference" "#PWR024" (at 106.68 148.59 0)
+    (property "Reference" "#PWR056" (at 106.68 148.59 0)
       (effects (font (size 1.27 1.27)) hide)
     )
@@
   (symbol (lib_id "power:GND") (at 139.7 91.44 270) (unit 1)
     (in_bom yes) (on_board yes) (dnp no) (fields_autoplaced)
-    (property "Reference" "#PWR021" (at 133.35 91.44 0)
+    (property "Reference" "#PWR057" (at 133.35 91.44 0)
       (effects (font (size 1.27 1.27)) hide)
     )
@@
   (symbol (lib_id "Device:R") (at 99.06 104.14 90) (unit 1)
     (in_bom yes) (on_board yes) (dnp no) (fields_autoplaced)
-    (property "Reference" "R16" (at 99.06 97.79 90)
+    (property "Reference" "R26" (at 99.06 97.79 90)
       (effects (font (size 1.27 1.27)))
     )
@@
   (symbol (lib_id "Device:C") (at 106.68 138.43 0) (unit 1)
     (in_bom yes) (on_board yes) (dnp no) (fields_autoplaced)
-    (property "Reference" "C15" (at 110.49 137.16 0)
+    (property "Reference" "C32" (at 110.49 137.16 0)
       (effects (font (size 1.27 1.27)) (justify left))
     )
@@
   (symbol (lib_id "power:+5V") (at 179.07 91.44 0) (unit 1)
     (in_bom yes) (on_board yes) (dnp no) (fields_autoplaced)
-    (property "Reference" "#PWR051" (at 179.07 95.25 0)
+    (property "Reference" "#PWR061" (at 179.07 95.25 0)
       (effects (font (size 1.27 1.27)) hide)
     )
@@
   (symbol (lib_id "power:GND") (at 165.1 96.52 90) (unit 1)
     (in_bom yes) (on_board yes) (dnp no) (fields_autoplaced)
-    (property "Reference" "#PWR023" (at 171.45 96.52 0)
+    (property "Reference" "#PWR060" (at 171.45 96.52 0)
       (effects (font (size 1.27 1.27)) hide)
     )
@@
   (symbol (lib_id "power:+5V") (at 157.48 83.82 270) (unit 1)
     (in_bom yes) (on_board yes) (dnp no) (fields_autoplaced)
-    (property "Reference" "#PWR027" (at 153.67 83.82 0)
+    (property "Reference" "#PWR058" (at 153.67 83.82 0)
       (effects (font (size 1.27 1.27)) hide)
     )
@@
   (symbol (lib_id "Device:C") (at 102.87 113.03 0) (unit 1)
     (in_bom yes) (on_board yes) (dnp no) (fields_autoplaced)
-    (property "Reference" "C25" (at 106.68 111.76 0)
+    (property "Reference" "C31" (at 106.68 111.76 0)
       (effects (font (size 1.27 1.27)) (justify left))
     )
@@
   (symbol (lib_id "power:GND") (at 157.48 86.36 90) (unit 1)
     (in_bom yes) (on_board yes) (dnp no) (fields_autoplaced)
-    (property "Reference" "#PWR026" (at 163.83 86.36 0)
+    (property "Reference" "#PWR059" (at 163.83 86.36 0)
       (effects (font (size 1.27 1.27)) hide)
     )
@@
   (symbol (lib_id "Device:C") (at 114.3 113.03 0) (unit 1)
     (in_bom yes) (on_board yes) (dnp no)
-    (property "Reference" "C27" (at 118.11 111.76 0)
+    (property "Reference" "C33" (at 118.11 111.76 0)
       (effects (font (size 1.27 1.27)) (justify left))
     )
@@
   (symbol (lib_id "power:GND") (at 100.33 116.84 270) (unit 1)
     (in_bom yes) (on_board yes) (dnp no) (fields_autoplaced)
-    (property "Reference" "#PWR028" (at 93.98 116.84 0)
+    (property "Reference" "#PWR054" (at 93.98 116.84 0)
       (effects (font (size 1.27 1.27)) hide)
     )
@@
   (symbol (lib_id "Device:C") (at 125.73 113.03 0) (unit 1)
     (in_bom yes) (on_board yes) (dnp no)
-    (property "Reference" "C29" (at 129.54 111.76 0)
-      (effects (font (size 1.27 1.27)) (justify left))
-    )
+    (property "Reference" "C34" (at 129.54 111.76 0)
+      (effects (font (size 1.27 1.27)) (justify left))
+    )

Commit message: added pull up resistor values
Parts:
- R29: value R -> 50k
Changed lines of the file:
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@@
       (effects (font (size 1.27 1.27)) (justify left))
     )
-    (property "Value" "R" (at 181.61 96.52 0)
+    (property "Value" "50k" (at 181.61 96.52 0)
       (effects (font (size 1.27 1.27)) (justify left))
     )

Commit message: fixed pull up resistor values
Parts:
- R29: value 50k -> 30k
Changed lines of the file:
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@@
       (effects (font (size 1.27 1.27)) (justify left))
     )
-    (property "Value" "50k" (at 181.61 96.52 0)
+    (property "Value" "30k" (at 181.61 96.52 0)
       (effects (font (size 1.27 1.27)) (justify left))
     )

Commit message: added eeprom values
Parts:
- C31, C33, C34: value C -> 5.6nF
- C32: value C -> 100nF
- R26, R27, R28: value R -> 10k
Changed lines of the file:
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@@
       (effects (font (size 1.27 1.27)))
     )
-    (property "Value" "R" (at 110.49 90.17 90)
+    (property "Value" "10k" (at 110.49 90.17 90)
       (effects (font (size 1.27 1.27)))
     )
@@
       (effects (font (size 1.27 1.27)))
     )
-    (property "Value" "R" (at 121.92 78.74 90)
+    (property "Value" "10k" (at 121.92 78.74 90)
       (effects (font (size 1.27 1.27)))
     )
@@
       (effects (font (size 1.27 1.27)))
     )
-    (property "Value" "R" (at 99.06 100.33 90)
+    (property "Value" "10k" (at 99.06 100.33 90)
       (effects (font (size 1.27 1.27)))
     )
@@
       (effects (font (size 1.27 1.27)) (justify left))
     )
-    (property "Value" "C" (at 110.49 139.7 0)
+    (property "Value" "100nF" (at 110.49 139.7 0)
       (effects (font (size 1.27 1.27)) (justify left))
     )
@@
       (effects (font (size 1.27 1.27)) (justify left))
     )
-    (property "Value" "C" (at 106.68 114.3 0)
+    (property "Value" "5.6nF" (at 106.68 114.3 0)
       (effects (font (size 1.27 1.27)) (justify left))
     )
@@
       (effects (font (size 1.27 1.27)) (justify left))
     )
-    (property "Value" "C" (at 118.11 114.3 0)
+    (property "Value" "5.6nF" (at 118.11 114.3 0)
       (effects (font (size 1.27 1.27)) (justify left))
     )
@@
       (effects (font (size 1.27 1.27)) (justify left))
     )
-    (property "Value" "C" (at 129.54 114.3 0)
-      (effects (font (size 1.27 1.27)) (justify left))
-    )
+    (property "Value" "5.6nF" (at 129.54 114.3 0)
+      (effects (font (size 1.27 1.27)) (justify left))
+    )

Commit message: renamed motor magic file
Parts:
- renumbered C31 to C5, C32 to C6, C33 to C7, C34 to C8, R26 to R4, R27 to R5, R28 to R6, R29 to R7, U8 to U3

Commit message: added LEDS and fuses
Parts:
- renumbered C5 to C31, C6 to C32, C7 to C33, C8 to C34, R4 to R26, R5 to R27, R6 to R28, R7 to R29, U3 to U8
Changed lines of the file:
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@@
   (symbol (lib_id "Device:R") (at 110.49 93.98 90) (unit 1)
     (in_bom yes) (on_board yes) (dnp no) (fields_autoplaced)
-    (property "Reference" "R5" (at 110.49 87.63 90)
+    (property "Reference" "R27" (at 110.49 87.63 90)
       (effects (font (size 1.27 1.27)))
     )
@@
   (symbol (lib_id "power:+5V") (at 106.68 134.62 0) (unit 1)
     (in_bom yes) (on_board yes) (dnp no) (fields_autoplaced)
-    (property "Reference" "#PWR010" (at 106.68 138.43 0)
+    (property "Reference" "#PWR055" (at 106.68 138.43 0)
       (effects (font (size 1.27 1.27)) hide)
     )
@@
   (symbol (lib_id "2022-lsd:AT28C64B") (at 148.59 99.06 0) (unit 1)
     (in_bom yes) (on_board yes) (dnp no) (fields_autoplaced)
-    (property "Reference" "U3" (at 148.59 76.2 0)
+    (property "Reference" "U8" (at 148.59 76.2 0)
       (effects (font (size 1.27 1.27)))
     )
@@
   (symbol (lib_id "Device:R") (at 179.07 95.25 0) (unit 1)
     (in_bom yes) (on_board yes) (dnp no) (fields_autoplaced)
-    (property "Reference" "R7" (at 181.61 93.98 0)
+    (property "Reference" "R29" (at 181.61 93.98 0)
       (effects (font (size 1.27 1.27)) (justify left))
     )
@@
   (symbol (lib_id "Device:R") (at 121.92 82.55 90) (unit 1)
     (in_bom yes) (on_board yes) (dnp no) (fields_autoplaced)
-    (property "Reference" "R6" (at 121.92 76.2 90)
+    (property "Reference" "R28" (at 121.92 76.2 90)
       (effects (font (size 1.27 1.27)))
     )
@@
   (symbol (lib_id "power:GND") (at 106.68 142.24 0) (unit 1)
     (in_bom yes) (on_board yes) (dnp no) (fields_autoplaced)
-    (property "Reference" "#PWR011" (at 106.68 148.59 0)
+    (property "Reference" "#PWR056" (at 106.68 148.59 0)
       (effects (font (size 1.27 1.27)) hide)
     )
@@
   (symbol (lib_id "power:GND") (at 139.7 91.44 270) (unit 1)
     (in_bom yes) (on_board yes) (dnp no) (fields_autoplaced)
-    (property "Reference" "#PWR012" (at 133.35 91.44 0)
+    (property "Reference" "#PWR057" (at 133.35 91.44 0)
       (effects (font (size 1.27 1.27)) hide)
     )
@@
   (symbol (lib_id "Device:R") (at 99.06 104.14 90) (unit 1)
     (in_bom yes) (on_board yes) (dnp no) (fields_autoplaced)
-    (property "Reference" "R4" (at 99.06 97.79 90)
+    (property "Reference" "R26" (at 99.06 97.79 90)
       (effects (font (size 1.27 1.27)))
     )
@@
   (symbol (lib_id "Device:C") (at 106.68 138.43 0) (unit 1)
     (in_bom yes) (on_board yes) (dnp no) (fields_autoplaced)
-    (property "Reference" "C6" (at 110.49 137.16 0)
+    (property "Reference" "C32" (at 110.49 137.16 0)
       (effects (font (size 1.27 1.27)) (justify left))
     )
@@
   (symbol (lib_id "power:+5V") (at 179.07 91.44 0) (unit 1)
     (in_bom yes) (on_board yes) (dnp no) (fields_autoplaced)
-    (property "Reference" "#PWR016" (at 179.07 95.25 0)
+    (property "Reference" "#PWR061" (at 179.07 95.25 0)
       (effects (font (size 1.27 1.27)) hide)
     )
@@
   (symbol (lib_id "power:GND") (at 165.1 96.52 90) (unit 1)
     (in_bom yes) (on_board yes) (dnp no) (fields_autoplaced)
-    (property "Reference" "#PWR015" (at 171.45 96.52 0)
+    (property "Reference" "#PWR060" (at 171.45 96.52 0)
       (effects (font (size 1.27 1.27)) hide)
     )
@@
   (symbol (lib_id "power:+5V") (at 157.48 83.82 270) (unit 1)
     (in_bom yes) (on_board yes) (dnp no) (fields_autoplaced)
-    (property "Reference" "#PWR013" (at 153.67 83.82 0)
+    (property "Reference" "#PWR058" (at 153.67 83.82 0)
       (effects (font (size 1.27 1.27)) hide)
     )
@@
   (symbol (lib_id "Device:C") (at 102.87 113.03 0) (unit 1)
     (in_bom yes) (on_board yes) (dnp no) (fields_autoplaced)
-    (property "Reference" "C5" (at 106.68 111.76 0)
+    (property "Reference" "C31" (at 106.68 111.76 0)
       (effects (font (size 1.27 1.27)) (justify left))
     )
@@
   (symbol (lib_id "power:GND") (at 157.48 86.36 90) (unit 1)
     (in_bom yes) (on_board yes) (dnp no) (fields_autoplaced)
-    (property "Reference" "#PWR014" (at 163.83 86.36 0)
+    (property "Reference" "#PWR059" (at 163.83 86.36 0)
       (effects (font (size 1.27 1.27)) hide)
     )
@@
   (symbol (lib_id "Device:C") (at 114.3 113.03 0) (unit 1)
     (in_bom yes) (on_board yes) (dnp no)
-    (property "Reference" "C7" (at 118.11 111.76 0)
+    (property "Reference" "C33" (at 118.11 111.76 0)
       (effects (font (size 1.27 1.27)) (justify left))
     )
@@
   (symbol (lib_id "power:GND") (at 100.33 116.84 270) (unit 1)
     (in_bom yes) (on_board yes) (dnp no) (fields_autoplaced)
-    (property "Reference" "#PWR09" (at 93.98 116.84 0)
+    (property "Reference" "#PWR054" (at 93.98 116.84 0)
       (effects (font (size 1.27 1.27)) hide)
     )
@@
   (symbol (lib_id "Device:C") (at 125.73 113.03 0) (unit 1)
     (in_bom yes) (on_board yes) (dnp no)
-    (property "Reference" "C8" (at 129.54 111.76 0)
-      (effects (font (size 1.27 1.27)) (justify left))
-    )
+    (property "Reference" "C34" (at 129.54 111.76 0)
+      (effects (font (size 1.27 1.27)) (justify left))
+    )
