File: main_board/kicad/stepDown-24-5.kicad_sch (KiCad schematic)
At the start: 5 parts, among them U1 LM2576S-5

Commit message: added hierarchy for 15v stepdown
Parts:
- removed C2: C, symbol Device:C
- added C2: C_Polarized, symbol Device:C_Polarized
Connections:
- net GND: now also C2.2
- net OUT renamed +5V
- net +5V: now also C2.1
Changed lines of the file:
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@@
     (stroke (width 0) (type default))
   )
-  (hierarchical_label "OUT" (shape output) (at 176.53 100.33 0) (fields_autoplaced)
-    (effects (font (size 1.27 1.27)) (justify left))
+  (symbol (lib_id "power:+5V") (at 176.53 100.33 270) (unit 1)
+    (in_bom yes) (on_board yes) (dnp no) (fields_autoplaced)
+    (property "Reference" "#PWR017" (at 172.72 100.33 0)
+      (effects (font (size 1.27 1.27)) hide)
+    )
+    (property "Value" "+5V" (at 180.34 100.33 90)
+      (effects (font (size 1.27 1.27)) (justify left))
+    )
+    (property "Footprint" "" (at 176.53 100.33 0)
+      (effects (font (size 1.27 1.27)) hide)
+    )
+    (property "Datasheet" "" (at 176.53 100.33 0)
+      (effects (font (size 1.27 1.27)) hide)
+    )
+    (pin "1")
+    (instances
+      (project "main"
+        (path "/9139d8e7-a5dc-421f-9a12-f77d83384a16/5ff0ce27-8c4e-4301-96f8-e492b23285ac"
+          (reference "#PWR017") (unit 1)
+        )
+      )
+    )
   )
   (symbol (lib_id "Diode:1N5822") (at 160.02 104.14 270) (unit 1)
@@
         (path "/9139d8e7-a5dc-421f-9a12-f77d83384a16/5ff0ce27-8c4e-4301-96f8-e492b23285ac"
           (reference "D1") (unit 1)
+        )
+      )
+    )
+  )
+  (symbol (lib_id "Device:C_Polarized") (at 173.99 104.14 0) (unit 1)
+    (in_bom yes) (on_board yes) (dnp no) (fields_autoplaced)
+    (property "Reference" "C2" (at 177.8 101.981 0)
+      (effects (font (size 1.27 1.27)) (justify left))
+    )
+    (property "Value" "C_Polarized" (at 177.8 104.521 0)
+      (effects (font (size 1.27 1.27)) (justify left))
+    )
+    (property "Footprint" "" (at 174.9552 107.95 0)
+      (effects (font (size 1.27 1.27)) hide)
+    )
+    (property "Datasheet" "~" (at 173.99 104.14 0)
+      (effects (font (size 1.27 1.27)) hide)
+    )
+    (pin "1")
+    (pin "2")
+    (instances
+      (project "main"
+        (path "/9139d8e7-a5dc-421f-9a12-f77d83384a16/5ff0ce27-8c4e-4301-96f8-e492b23285ac"
+          (reference "C2") (unit 1)
         )
       )
@@
         )
       )
-    )
-  )
-  (symbol (lib_id "Device:C") (at 173.99 104.14 0) (unit 1)
-    (in_bom yes) (on_board yes) (dnp no)
-    (property "Reference" "C2" (at 177.8 102.8699 90)
-      (effects (font (size 1.27 1.27)) (justify left))
-    )
-    (property "Value" "C" (at 177.8 105.4099 0)
-      (effects (font (size 1.27 1.27)) (justify left))
-    )
-    (property "Footprint" "" (at 174.9552 107.95 0)
-      (effects (font (size 1.27 1.27)) hide)
-    )
-    (property "Datasheet" "~" (at 173.99 104.14 0)
-      (effects (font (size 1.27 1.27)) hide)
-    )
-    (pin "1")
-    (pin "2")
-    (instances
-      (project "main"
-        (path "/9139d8e7-a5dc-421f-9a12-f77d83384a16"
-          (reference "C2") (unit 1)
-        )
-        (path "/9139d8e7-a5dc-421f-9a12-f77d83384a16/5ff0ce27-8c4e-4301-96f8-e492b23285ac"
-          (reference "C2") (unit 1)
-        )
-      )

Commit message: added first capacitor value for stepdown
Parts:
- C1: value C -> 100nF
Changed lines of the file:
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@@
       (effects (font (size 1.27 1.27)) (justify left))
     )
-    (property "Value" "C" (at 123.19 101.5999 0)
+    (property "Value" "100nF" (at 123.19 101.5999 0)
       (effects (font (size 1.27 1.27)) (justify left))
     )

Commit message: added LEDS and fuses
Parts:
- added F1: Fuse 1A, symbol Device:Fuse
- C2: value C_Polarized -> 1000uF
- L1: value L -> 150uH
Connections:
- net +5V: now also F1.2; no longer C2.1, L1.2, U1.4 (FB)
- new net: C2.1, F1.1, L1.2, U1.4 (FB)
Changed lines of the file:
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@@
     (stroke (width 0) (type default))
   )
-  (wire (pts (xy 173.99 100.33) (xy 176.53 100.33))
+  (wire (pts (xy 173.99 100.33) (xy 180.34 100.33))
     (stroke (width 0) (type default))
   )
-  (symbol (lib_id "power:+5V") (at 176.53 100.33 270) (unit 1)
-    (in_bom yes) (on_board yes) (dnp no) (fields_autoplaced)
-    (property "Reference" "#PWR017" (at 172.72 100.33 0)
-      (effects (font (size 1.27 1.27)) hide)
-    )
-    (property "Value" "+5V" (at 180.34 100.33 90)
-      (effects (font (size 1.27 1.27)) (justify left))
-    )
-    (property "Footprint" "" (at 176.53 100.33 0)
-      (effects (font (size 1.27 1.27)) hide)
-    )
-    (property "Datasheet" "" (at 176.53 100.33 0)
+  (symbol (lib_id "power:+5V") (at 187.96 100.33 270) (unit 1)
+    (in_bom yes) (on_board yes) (dnp no) (fields_autoplaced)
+    (property "Reference" "#PWR017" (at 184.15 100.33 0)
+      (effects (font (size 1.27 1.27)) hide)
+    )
+    (property "Value" "+5V" (at 191.77 100.33 90)
+      (effects (font (size 1.27 1.27)) (justify left))
+    )
+    (property "Footprint" "" (at 187.96 100.33 0)
+      (effects (font (size 1.27 1.27)) hide)
+    )
+    (property "Datasheet" "" (at 187.96 100.33 0)
       (effects (font (size 1.27 1.27)) hide)
     )
@@
     )
   )
+  (symbol (lib_id "Device:Fuse") (at 184.15 100.33 90) (unit 1)
+    (in_bom yes) (on_board yes) (dnp no) (fields_autoplaced)
+    (property "Reference" "F1" (at 184.15 95.25 90)
+      (effects (font (size 1.27 1.27)))
+    )
+    (property "Value" "Fuse 1A" (at 184.15 97.79 90)
+      (effects (font (size 1.27 1.27)))
+    )
+    (property "Footprint" "" (at 184.15 102.108 90)
+      (effects (font (size 1.27 1.27)) hide)
+    )
+    (property "Datasheet" "~" (at 184.15 100.33 0)
+      (effects (font (size 1.27 1.27)) hide)
+    )
+    (pin "1")
+    (pin "2")
+    (instances
+      (project "main"
+        (path "/9139d8e7-a5dc-421f-9a12-f77d83384a16/5ff0ce27-8c4e-4301-96f8-e492b23285ac"
+          (reference "F1") (unit 1)
+        )
+      )
+    )
+  )
   (symbol (lib_id "Diode:1N5822") (at 160.02 104.14 270) (unit 1)
     (in_bom yes) (on_board yes) (dnp no) (fields_autoplaced)
@@
       (effects (font (size 1.27 1.27)) (justify left))
     )
-    (property "Value" "C_Polarized" (at 177.8 104.521 0)
+    (property "Value" "1000uF" (at 177.8 104.521 0)
       (effects (font (size 1.27 1.27)) (justify left))
     )
@@
       (effects (font (size 1.27 1.27)))
     )
-    (property "Value" "L" (at 166.37 96.52 90)
-      (effects (font (size 1.27 1.27)))
-    )
+    (property "Value" "150uH" (at 166.37 96.52 90)
+      (effects (font (size 1.27 1.27)))
+    )

Commit message: resolved ERC
Changed lines of the file:
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@@
   (junction (at 143.51 107.95) (diameter 0) (color 0 0 0 0)
   )
+  (junction (at 127 95.25) (diameter 0) (color 0 0 0 0)
+  )
   (junction (at 173.99 100.33) (diameter 0) (color 0 0 0 0)
   )
@@
     (stroke (width 0) (type default))
   )
+  (wire (pts (xy 127 95.25) (xy 119.38 95.25))
+    (stroke (width 0) (type default))
+  )
   (wire (pts (xy 156.21 100.33) (xy 160.02 100.33))
     (stroke (width 0) (type default))
   )
-  (wire (pts (xy 130.81 95.25) (xy 119.38 95.25))
+  (wire (pts (xy 130.81 95.25) (xy 127 95.25))
     (stroke (width 0) (type default))
   )
@@
         )
       )
+    )
+  )
+  (symbol (lib_id "power:PWR_FLAG") (at 127 95.25 0) (unit 1)
+    (in_bom yes) (on_board yes) (dnp no) (fields_autoplaced)
+    (property "Reference" "#FLG03" (at 127 93.345 0)
+      (effects (font (size 1.27 1.27)) hide)
+    )
+    (property "Value" "PWR_FLAG" (at 127 90.17 0)
+      (effects (font (size 1.27 1.27)))
+    )
+    (property "Footprint" "" (at 127 95.25 0)
+      (effects (font (size 1.27 1.27)) hide)
+    )
+    (property "Datasheet" "~" (at 127 95.25 0)
+      (effects (font (size 1.27 1.27)) hide)
+    )
+    (pin "1")
+    (instances
+      (project "main"
+        (path "/9139d8e7-a5dc-421f-9a12-f77d83384a16/5ff0ce27-8c4e-4301-96f8-e492b23285ac"
+          (reference "#FLG03") (unit 1)
+        )
+      )

Commit message: added probe point
Parts:
- added TP1 (x2): TestPoint_Probe, symbol Connector:TestPoint_Probe
Connections:
- net +5V: now also TP1.1
- net GND: now also TP1.1
Changed lines of the file:
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@@
   (junction (at 119.38 95.25) (diameter 0) (color 0 0 0 0)
   )
+  (junction (at 189.738 100.33) (diameter 0) (color 0 0 0 0)
+  )
   (junction (at 130.81 107.95) (diameter 0) (color 0 0 0 0)
   )
@@
   (junction (at 127 95.25) (diameter 0) (color 0 0 0 0)
   )
+  (junction (at 149.098 107.95) (diameter 0) (color 0 0 0 0)
+  )
   (junction (at 173.99 100.33) (diameter 0) (color 0 0 0 0)
   )
@@
     (stroke (width 0) (type default))
   )
+  (wire (pts (xy 149.098 107.95) (xy 143.51 107.95))
+    (stroke (width 0) (type default))
+  )
   (wire (pts (xy 160.02 107.95) (xy 173.99 107.95))
     (stroke (width 0) (type default))
@@
     (stroke (width 0) (type default))
   )
-  (wire (pts (xy 160.02 107.95) (xy 143.51 107.95))
+  (wire (pts (xy 160.02 107.95) (xy 149.098 107.95))
     (stroke (width 0) (type default))
   )
@@
     (stroke (width 0) (type default))
   )
+  (wire (pts (xy 189.738 100.33) (xy 187.96 100.33))
+    (stroke (width 0) (type default))
+  )
   (wire (pts (xy 173.99 100.33) (xy 180.34 100.33))
     (stroke (width 0) (type default))
   )
-  (symbol (lib_id "power:+5V") (at 187.96 100.33 270) (unit 1)
+  (wire (pts (xy 191.008 100.33) (xy 189.738 100.33))
+    (stroke (width 0) (type default))
+  )
+  (symbol (lib_id "Connector:TestPoint_Probe") (at 149.098 107.95 0) (unit 1)
+    (in_bom yes) (on_board yes) (dnp no)
+    (property "Reference" "TP1" (at 146.304 109.982 0)
+      (effects (font (size 1.27 1.27)) (justify left))
+    )
+    (property "Value" "TestPoint_Probe" (at 146.304 112.014 0)
+      (effects (font (size 1.27 1.27)) (justify left))
+    )
+    (property "Footprint" "" (at 154.178 107.95 0)
+      (effects (font (size 1.27 1.27)) hide)
+    )
+    (property "Datasheet" "~" (at 154.178 107.95 0)
+      (effects (font (size 1.27 1.27)) hide)
+    )
+    (pin "1")
+    (instances
+      (project "main"
+        (path "/9139d8e7-a5dc-421f-9a12-f77d83384a16/4605f0e7-6d1c-410b-b12b-1c5d8b870a3a"
+          (reference "TP1") (unit 1)
+        )
+        (path "/9139d8e7-a5dc-421f-9a12-f77d83384a16/5ff0ce27-8c4e-4301-96f8-e492b23285ac"
+          (reference "TP4") (unit 1)
+        )
+      )
+    )
+  )
+  (symbol (lib_id "power:+5V") (at 191.008 100.33 270) (unit 1)
     (in_bom yes) (on_board yes) (dnp no) (fields_autoplaced)
-    (property "Reference" "#PWR017" (at 184.15 100.33 0)
-      (effects (font (size 1.27 1.27)) hide)
-    )
-    (property "Value" "+5V" (at 191.77 100.33 90)
-      (effects (font (size 1.27 1.27)) (justify left))
-    )
-    (property "Footprint" "" (at 187.96 100.33 0)
-      (effects (font (size 1.27 1.27)) hide)
-    )
-    (property "Datasheet" "" (at 187.96 100.33 0)
+    (property "Reference" "#PWR017" (at 187.198 100.33 0)
+      (effects (font (size 1.27 1.27)) hide)
+    )
+    (property "Value" "+5V" (at 194.818 100.33 90)
+      (effects (font (size 1.27 1.27)) (justify left))
+    )
+    (property "Footprint" "" (at 191.008 100.33 0)
+      (effects (font (size 1.27 1.27)) hide)
+    )
+    (property "Datasheet" "" (at 191.008 100.33 0)
       (effects (font (size 1.27 1.27)) hide)
     )
@@
         )
       )
+    )
+  )
+  (symbol (lib_id "Connector:TestPoint_Probe") (at 189.738 100.33 0) (unit 1)
+    (in_bom yes) (on_board yes) (dnp no)
+    (property "Reference" "TP1" (at 186.944 102.362 0)
+      (effects (font (size 1.27 1.27)) (justify left))
+    )
+    (property "Value" "TestPoint_Probe" (at 186.944 104.394 0)
+      (effects (font (size 1.27 1.27)) (justify left))
+    )
+    (property "Footprint" "" (at 194.818 100.33 0)
+      (effects (font (size 1.27 1.27)) hide)
+    )
+    (property "Datasheet" "~" (at 194.818 100.33 0)
+      (effects (font (size 1.27 1.27)) hide)
+    )
+    (pin "1")
+    (instances
+      (project "main"
+        (path "/9139d8e7-a5dc-421f-9a12-f77d83384a16/4605f0e7-6d1c-410b-b12b-1c5d8b870a3a"
+          (reference "TP1") (unit 1)
+        )
+        (path "/9139d8e7-a5dc-421f-9a12-f77d83384a16/5ff0ce27-8c4e-4301-96f8-e492b23285ac"
+          (reference "TP3") (unit 1)
+        )
+      )

Commit message: updated to post review state
Parts:
- removed C1: 100nF, symbol Device:C
- removed TP1 (x2): TestPoint_Probe, symbol Connector:TestPoint_Probe
- added C23: 100uF, symbol Device:C_Polarized
- added TP1, TP2: TestPoint_Probe, symbol Connector:TestPoint_Probe
Connections:
- net +24V: now also F1.2; no longer U1.1 (VIN)
- net +5V: now also C2.1, L1.2, U1.4 (FB), TP1.1; no longer F1.2
- net GND: now also C23.2, TP2.1
- new net: C23.1, F1.1, U1.1 (VIN)
Other:
- moved on the sheet: F1

Commit message: added footprints
Parts:
- C2: footprint (none) -> Capacitor_THT:CP_Radial_D10.0mm_P5.00mm
- C23: footprint (none) -> Capacitor_THT:CP_Radial_D6.3mm_P2.50mm
- F1: footprint (none) -> Fuse:Fuseholder_Cylinder-5x20mm_Schurter_0031_8201_Horizontal_Open
- L1: footprint (none) -> Inductor_THT:L_Radial_D12.5mm_P7.00mm_Fastron_09HCP
- TP1, TP2: footprint (none) -> TestPoint:TestPoint_Pad_D3.0mm
Changed lines of the file:
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@@
       (effects (font (size 1.27 1.27)) (justify left))
     )
-    (property "Footprint" "" (at 152.4 107.95 0)
+    (property "Footprint" "TestPoint:TestPoint_Pad_D3.0mm" (at 152.4 107.95 0)
       (effects (font (size 1.27 1.27)) hide)
     )
@@
       (effects (font (size 1.27 1.27)) (justify right))
     )
-    (property "Footprint" "" (at 121.158 82.55 90)
+    (property "Footprint" "Fuse:Fuseholder_Cylinder-5x20mm_Schurter_0031_8201_Horizontal_Open" (at 121.158 82.55 90)
       (effects (font (size 1.27 1.27)) hide)
     )
@@
       (effects (font (size 1.27 1.27)) (justify left))
     )
-    (property "Footprint" "" (at 174.9552 107.95 0)
+    (property "Footprint" "Capacitor_THT:CP_Radial_D10.0mm_P5.00mm" (at 174.9552 107.95 0)
       (effects (font (size 1.27 1.27)) hide)
     )
@@
       (effects (font (size 1.27 1.27)) (justify left))
     )
-    (property "Footprint" "" (at 120.3452 104.14 0)
+    (property "Footprint" "Capacitor_THT:CP_Radial_D6.3mm_P2.50mm" (at 120.3452 104.14 0)
       (effects (font (size 1.27 1.27)) hide)
     )
@@
       (effects (font (size 1.27 1.27)) (justify left))
     )
-    (property "Footprint" "" (at 181.61 100.33 0)
+    (property "Footprint" "TestPoint:TestPoint_Pad_D3.0mm" (at 181.61 100.33 0)
       (effects (font (size 1.27 1.27)) hide)
     )
@@
       (effects (font (size 1.27 1.27)))
     )
-    (property "Footprint" "" (at 166.37 100.33 0)
-      (effects (font (size 1.27 1.27)) hide)
-    )
+    (property "Footprint" "Inductor_THT:L_Radial_D12.5mm_P7.00mm_Fastron_09HCP" (at 166.37 100.33 0)
+      (effects (font (size 1.27 1.27)) hide)
+    )
