File: main_board/kicad/stepDown-24-5.kicad_sch (KiCad schematic)
At the start: 8 parts, among them U1 LM2576S-5

Commit message: implemented bridge and first bridge driver as well as both step converters on the pcd layout
Parts:
- U1: footprint Package_TO_SOT_SMD:TO-263-5_TabPin3 -> Package_TO_SOT_THT:TO-220-5_Vertical
Changed lines of the file:
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@@
       (effects (font (size 1.27 1.27)))
     )
-    (property "Footprint" "Package_TO_SOT_SMD:TO-263-5_TabPin3" (at 143.51 104.14 0)
+    (property "Footprint" "Package_TO_SOT_THT:TO-220-5_Vertical" (at 143.51 104.14 0)
       (effects (font (size 1.27 1.27) italic) (justify left) hide)
     )
