File: main_board/kicad/main.kicad_pcb (KiCad board)
At the start: 2 copper layers, 200 x 150 mm, 148 parts, among them J1 Sensorbuchse, J2 Motorbuchse, J3 Motorbuchse, J4 Batteriebuchse, J5 Conn_02x07_Odd_Even, J6 Sensorbuchse, J7 AVR-ISP-10, Q1 IRFB3077, Q13 IRFB3077, Q14 IRFB3077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

Commit message: moved logic sockets
Parts:
- moved D27 134.7 mm to (141.1, -0.86)
- moved D28 134.7 mm to (154.2, -8.74)
- moved D29 134.7 mm to (161.7, -8.74)
- moved D30 134.7 mm to (169.2, -8.74)
- moved R50 134.7 mm to (136.1, -11.2)
- moved R51 134.7 mm to (159.8, 1.27)
- moved R52 134.7 mm to (159.0, -20.8)
- moved R53 134.7 mm to (169.9, 1.52)
- moved R24 10.8 mm to (221.2, 126.7), turned to -90 degrees
- moved R21 6.48 mm to (207.5, 53.7)
- moved C16 3.74 mm to (219.7, 103.4)
- moved R23 3.23 mm to (196.6, 136.4)
- moved U5 1.66 mm to (201.4, 98.8)
- moved U8 0.63 mm to (201.4, 59.7)
Routing:
- net /MotorMagic_R/HAL2: track 387.7 -> 378.5 mm
- net /MotorMagic_L/HAL1: track 155.1 -> 149.9 mm
- net /MotorMagic_L/bridgeDriver2/G_L_IN: track 60.6 -> 65.1 mm
- net Net-(U8-A1): track 24.1 -> 19.9 mm
- net /MotorMagic_R/HAL3: track 366.1 -> 370.0 mm
- net /DIR_L_REG: track 313.5 -> 310.3 mm
- net +5V: track 891.1 -> 888.1 mm
- net Net-(U8-A2): track 25.5 -> 22.8 mm
- net /PWM_R_REG: track 230.9 -> 233.3 mm
- net GND: track 1472.1 -> 1469.7 mm
- net Net-(U5-A2): track 58.0 -> 60.2 mm
- net /MotorMagic_R/bridgeDriver2/Y_H_IN: track 72.1 -> 70.3 mm
- net /MotorMagic_L/bridgeDriver2/B_L_IN: track 63.5 -> 61.7 mm
- net /DIR_R_REG: track 230.7 -> 232.4 mm
- net /MotorMagic_R/bridgeDriver2/B_H_IN: track 77.9 -> 76.2 mm
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Other:
- board text added: "1 Möhring'scher Normabstand"

Commit message: optimization
Parts:
- moved D29 171.9 mm to (1.27, 53.1), turned to 90 degrees
- moved D28 167.9 mm to (1.27, 60.6), turned to 90 degrees
- moved R52 167.3 mm to (4.93, 44.3), turned to 90 degrees
- moved D30 160.6 mm to (12.0, 24.5), turned to 90 degrees
- moved D27 151.5 mm to (9.14, 73.7), turned to 90 degrees
- moved R53 148.2 mm to (23.9, 26.7), turned to 90 degrees
- moved R51 147.3 mm to (18.1, 41.8), turned to -90 degrees
- moved R50 143.1 mm to (13.6, 62.6), turned to 90 degrees
- moved C35 13.2 mm to (204.5, 34.9), turned to 90 degrees
- moved C21 9.67 mm to (161.3, 33.7), turned to 180 degrees
- moved C36 8.01 mm to (210.8, 27.9), turned to 180 degrees
Routing:
- net /attiny13/SCK: track 160.1 -> 18.5 mm
- net /MotorMagic_R/G_OUT: track 137.9 -> 203.4 mm, vias 1 -> 0
- net /MotorMagic_L/HAL2: track 210.6 -> 170.0 mm
- net /attiny13/Battery_Charge_PWM: track 229.6 -> 269.1 mm
- net /MotorMagic_L/HAL3: track 205.5 -> 178.9 mm
- net /MotorMagic_R/HAL1: track 409.8 -> 389.8 mm
- net /MotorMagic_R/B_OUT: track 144.5 -> 133.0 mm
- net /ENABLE_L_REG: track 199.3 -> 188.0 mm
- net /attiny13//RESET: track 183.1 -> 171.9 mm
- net /MotorMagic_R/HAL3: track 370.0 -> 359.3 mm
- net /MotorMagic_L/Y_OUT: track 173.6 -> 182.7 mm
- net /DIR_L_REG: track 310.3 -> 316.8 mm, vias 2 -> 0
- net +15V: track 300.6 -> 307.0 mm
- net /MotorMagic_R/HAL2: track 378.5 -> 373.9 mm
- net /MotorMagic_L/bridge2/B_H: track 92.6 -> 89.4 mm
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