File: main_board/kicad/main.kicad_pcb (KiCad board)
At the start: 2 copper layers, 200 x 150 mm, 148 parts, among them J1 Sensorbuchse, J2 Motorbuchse, J3 Motorbuchse, J4 Batteriebuchse, J5 Conn_02x07_Odd_Even, J6 Sensorbuchse, J7 AVR-ISP-10, Q1 IRFB3077, Q13 IRFB3077, Q14 IRFB3077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

Commit message: more optimization
Parts:
- moved D28 189.0 mm to (186.9, 25.4), turned to 180 degrees
- moved D27 174.5 mm to (157.0, 166.4)
- moved R50 169.9 mm to (153.2, 159.5), turned to 0 degrees
- moved R51 163.8 mm to (181.1, 25.4), turned to 180 degrees
- moved D7 21.9 mm to (143.8, 145.3), turned to -90 degrees
- moved R14 19.8 mm to (166.9, 155.7)
- moved R6 17.6 mm to (138.9, 159.0)
- moved R11 13.2 mm to (166.9, 152.4)
- moved R13 13.2 mm to (166.9, 139.2)
- moved C41 12.0 mm to (65.6, 97.0), turned to 0 degrees
- moved C42 12.0 mm to (121.5, 97.0), turned to 0 degrees
- moved C40 12.0 mm to (93.5, 97.0), turned to 0 degrees
- moved C5 11.7 mm to (70.0, 111.3), turned to 180 degrees
- moved C6 11.7 mm to (98.0, 111.3), turned to 180 degrees
- moved C7 11.7 mm to (125.9, 111.3), turned to 180 degrees
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Routing:
- net /attiny13/SCK: track 18.5 -> 184.4 mm
- net GND: track 1467.8 -> 1358.7 mm
- net +15V: track 307.0 -> 376.4 mm
- net /DIR_L_REG: track 316.8 -> 248.2 mm
- net +5V: track 889.4 -> 824.0 mm
- net /MotorMagic_R/G_OUT: track 203.4 -> 140.9 mm
- net /MotorMagic_R/bridge2/Y_H: track 101.3 -> 62.4 mm
- net +24V: track 219.4 -> 252.6 mm
- net /MotorMagic_L/bridge2/G_L: track 105.0 -> 135.4 mm, vias 1 -> 0
- net /MotorMagic_R/bridge2/Y_L: track 115.1 -> 89.7 mm, vias 1 -> 0
- net Net-(U3-HO1): track 45.8 -> 21.2 mm
- net /MotorMagic_R/bridge2/G_H: track 125.9 -> 103.9 mm, vias 1 -> 0
- net /MotorMagic_L/Y_OUT: track 182.7 -> 165.5 mm
- net /MotorMagic_L/B_OUT: track 100.7 -> 116.9 mm, vias 2 -> 1
- net /MotorMagic_L/HAL1: track 150.3 -> 135.1 mm
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- added copper zone on B.Cu, net GND
- removed copper zone on F.Cu, net GND
Other:
- board text added: "E_L"
- board text added: "HAL_L"
- board text added: "HAL_R"
- board text added: "TODO"

Commit message: solved DRC
Parts:
- added G***: LOGO, LOGO, F.Cu at (99.8, 162.1)
- moved R52 227.7 mm to (212.6, 136.4), turned to 180 degrees
- moved D29 226.6 mm to (213.6, 140.0), turned to -90 degrees
- moved D30 186.2 mm to (195.6, 56.1), turned to -90 degrees
- moved R53 179.5 mm to (197.9, 70.9)
- moved R8 7.62 mm to (45.7, 166.4), turned to 0 degrees
- moved R38 7.38 mm to (74.7, 50.5), turned to 180 degrees
- moved R23 5.08 mm to (191.5, 136.4)
- moved R30 3.18 mm to (65.4, 38.1)
- moved D20 2.79 mm to (144.8, 63.8)
- moved C18 2.37 mm to (171.2, 52.1), turned to 180 degrees
- moved C14 1.15 mm to (170.2, 138.7)
- moved R42 0.36 mm to (148.8, 56.1)
Routing:
- net /MotorMagic_R/B_OUT: track 124.7 -> 251.7 mm
- net /MotorMagic_L/B_OUT: track 116.9 -> 242.6 mm
- net /MotorMagic_L/G_OUT: track 130.1 -> 243.5 mm, vias 1 -> 2
- net GND: track 1358.7 -> 1452.4 mm
- net /MotorMagic_R/G_OUT: track 140.9 -> 221.1 mm
- net /MotorMagic_R/Y_OUT: track 199.6 -> 244.3 mm
- net /MotorMagic_L/Y_OUT: track 165.5 -> 204.3 mm, vias 0 -> 1
- net +15V: track 376.4 -> 412.2 mm
- net /MotorMagic_L/bridge2/Y_H: track 69.7 -> 91.9 mm
- net /DIR_R_REG: track 232.4 -> 252.9 mm
- net /MotorMagic_L/HAL1: track 135.1 -> 149.8 mm
- net /MotorMagic_L/bridge2/B_L: track 58.3 -> 72.8 mm
- net /ENABLE_R_REG: track 300.0 -> 314.5 mm
- net /MotorMagic_R/HAL3: track 359.3 -> 347.9 mm
- net /DIR_L_REG: track 248.2 -> 259.5 mm
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Other:
- board text added: "DIR_L"
- board text added: "DIR_R"
- board text added: "ENA_L"
- board text added: "ENA_R"
- board text added: "LSD-GR4-LST-D-B"
- board text added: "LSD-GR4-LST-D-T"
- board text added: "LSD-GR4-LST-D-TSTOP"
- board text removed: "E_L"
- board text removed: "TODO"

Commit message: finalized board
Parts:
- added REF**: Heatsink_Fischer_SK487-SA_84x8mm_2xDrill3.5mm_ScrewM3, 2022-lsd:Heatsink_Fischer_SK487-SA_84x8mm_2xDrill3.5mm_ScrewM3, F.Cu at (47.1, 83.6)
- added REF**: Heatsink_Fischer_SK487-SA_84x8mm_2xDrill3.5mm_ScrewM3, 2022-lsd:Heatsink_Fischer_SK487-SA_84x8mm_2xDrill3.5mm_ScrewM3, F.Cu at (47.1, 134.2)
- moved C22 151.5 mm to (94.4, 31.4), turned to -90 degrees
- moved J4 1.63 mm to (38.1, 96.5)
- moved J2 1.27 mm to (38.1, 55.9)
- moved J3 1.27 mm to (38.1, 142.2)
- moved J6 0.77 mm to (219.8, 52.2)
- moved J5 0.49 mm to (47.0, 34.4)
- moved J1 0.27 mm to (219.8, 158.9)
Routing:
- net +15V: track 412.2 -> 425.6 mm
- net +5V: track 824.8 -> 837.6 mm
- net GND: track 1452.4 -> 1464.0 mm
- net /MotorMagic_R/B_OUT: track 251.7 -> 260.7 mm
- net /MotorMagic_L/B_OUT: track 242.6 -> 234.0 mm
- net /MotorMagic_L/bridge2/Y_H: track 91.9 -> 86.4 mm
- net /MotorMagic_L/Y_OUT: track 204.3 -> 209.4 mm
- net /attiny13/Battery_Charge_PWM: track 267.6 -> 262.9 mm
- net /MotorMagic_R/bridge2/Y_H: track 62.4 -> 66.9 mm
- net /MotorMagic_R/bridge2/B_L: track 161.7 -> 165.3 mm
- net /MotorMagic_L/bridge2/B_H: track 88.5 -> 85.5 mm
- net /DIR_L_REG: track 259.5 -> 261.7 mm
- net /MotorMagic_R/HAL2: track 372.2 -> 370.1 mm
- net /MotorMagic_R/HAL1: track 387.8 -> 385.8 mm
- net +24V: track 252.6 -> 254.1 mm
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